File: schematics/projects/climate sensor/lw_board.sch (EAGLE design)
At the start: 34 parts, among them J11 J4_FS_2, J3 J2, J7 KF301-5.0, J8 KF301-5.0, Q1 2N3904, Q2 2N3904, Q3 2N3904, Q4 2N3904, Q5 2N3904, Q6 2N3904, U1 BME280, U2 PMS7003, U3 ESP32 DEVKIT WROOM-32D

Commit message: rename elements, optimize board
Parts:
- removed GY_SGP30_1: GY-SGP30, my_devices:GY-SGP30
- added U5: BME280, my_devices:BME280
- R1: value 10K -> 600
- R11: value 30 -> 600
- R12: value 100 -> 600
- R14: value 10K -> 100
- R7: value 600 -> 30
- R8, R9: value 600 -> 10K
- U1: value BME280 -> GY-SGP30; device my_devices:BME280 -> my_devices:GY-SGP30
- U2: value PMS7003 -> ESP32 DEVKIT WROOM-32D; device my_devices:PMS7003 -> my_devices:ESP32
- U3: value ESP32 DEVKIT WROOM-32D -> PMS7003; device my_devices:ESP32 -> my_devices:PMS7003
- renumbered J11 to J12, J3 to J10, J7 to J5, J8 to J6, U$11 to U6, U$4 to U4, U$6 to D2
Connections:
- removed net N$23 (its old number): Q3.B, R6.P$2
- new net N$27: Q3.B, R10.P$2
- net +5V: now also Q4.C, Q5.C, Q6.C, R1.P$2, R14.P$1, R4.P$2, U2.5V, U3.VCC; no longer Q1.C, Q2.C, Q3.C, R10.P$2, R12.P$1, R9.P$2, U2.VCC, U3.5V
- net 3V3: now also R2.P$2, R5.P$2, R7.P$1, R8.P$1, R9.P$1, U1.VIN, U5.VCC; no longer GY_SGP30_1.VIN, R1.P$1, R11.P$1, R14.P$1, R7.P$2, R8.P$2, U1.VCC
- net GND: now also Q1.E, Q2.E, Q3.E, U5.GND; no longer GY_SGP30_1.GND, Q4.E, Q5.E, Q6.E
- net GPIO_AN_A: now also R3.P$2, U2.IO34; no longer R2.P$2, U3.IO34
- net GPIO_AN_B: now also R6.P$2, U2.IO35; no longer R3.P$2, U3.IO35
- net GPIO_IR: now also R10.P$1, U2.IO2; no longer R13.P$1, U3.IO2
- net GPIO_RGB_B: now also R11.P$1, U2.IO27; no longer R4.P$1, U3.IO27
- net GPIO_RGB_G: now also R12.P$1, U2.IO26; no longer R5.P$1, U3.IO26
- net GPIO_RGB_R: now also R13.P$1, U2.IO25; no longer R6.P$1, U3.IO25
- net GPIO_TS: now also U2.IO4; no longer U3.IO4
- net I2C_SCL: now also U2.IO23, U5.SCL; no longer GY_SGP30_1.SCL, U3.IO23
- net I2C_SDA: now also U2.IO21, U5.SDA; no longer GY_SGP30_1.SDA, U3.IO21
- net N$1: now also Q4.E; no longer Q1.E
- net N$11: now also U2.IO32; no longer U3.IO32
- net N$2: now also Q5.E; no longer Q2.E
- net N$21: now also Q4.B, R11.P$2; no longer Q1.B, R4.P$2
- net N$22: now also Q5.B, R12.P$2; no longer Q2.B, R5.P$2
- net N$24: now also R7.P$2, U2.3V3; no longer R11.P$2, U3.3V3
- net N$25: now also Q3.C; no longer Q6.C
- net N$26: now also R14.P$2; no longer R12.P$2
- net N$28: now also R9.P$2, U3.SET; no longer R14.P$2, U2.SET
- net N$3: now also Q6.E; no longer Q3.E
- net N$4: now also Q2.B, R4.P$1; no longer Q4.B, R10.P$1
- net N$5: now also Q1.B, R1.P$1; no longer Q5.B, R9.P$1
- net N$6: now also Q1.C, R3.P$1; no longer Q5.C, R7.P$1
- net N$7: now also Q2.C, R5.P$1, R6.P$1; no longer Q4.C, R3.P$1, R8.P$1
- net N$8: now also R8.P$2, U3.RESET; no longer R1.P$2, U2.RESET
- net UART_0_RXD: now also U2.RXD0; no longer U3.RXD0
- net UART_0_TXD: now also U2.TXD0; no longer U3.TXD0
- net UART_1_RXD: now also U2.SD2, U3.TXD; no longer U2.TXD, U3.SD2
- net UART_1_TXD: now also U2.SD3, U3.RXD; no longer U2.RXD, U3.SD3
Other:
- moved on the sheet: Q1, Q2, Q3, Q4, Q5, Q6, R1, R10, R11, R12, R13, R14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
