File: schematics/projects/window_control/full_schema.sch (EAGLE design)
At the start: 40 parts, among them IC1 MEGA32-P, J1 SERVO, Q4 2N3904, Q5 2N3904, Q6 2N3904, Q8 MOSFET_N, SW1 SWITCH, U1 ESP32, U2 5V, U3 3V3

Commit message: Added ability to recalibrate SGP30 sensor (on hot-replace for example to another module)
Parts:
- removed U$1, U$2: L, my_devices:L
- added BM1: EM-9767P, my_devices:MICROPHONE
- added C10, C9: 0.01uF, my_devices:C-1
- added C11, C12: 22pF, my_devices:C-1
- added C13, C14: 10pF, my_devices:C-1
- added C8: 33pF, my_devices:C-1
- added L1: L-3, my_devices:L-3
- added L2: L-2, my_devices:L-2
- added Q9: STP14NM50N, my_devices:MOSFET_N
- added R10: 200k, my_devices:R
- added R14, R15: 10K, my_devices:R
- added U4: GY-SGP30, my_devices:GY-SGP30
- added U5: BMP280, my_devices:BME280
- added U6: MSGEQ7, my_devices:MSGEQ7
- added U7: 433MHZ_TRANSMITTER, my_devices:433MHZ_TRANSMITTER
- added X1: HC-49S (16MHZ), my_devices:X
- C1, C2: value C -> K10-17B (1000pF)
- C3, C4, C5: value C -> 1000uF
- C6: value 0.1mkF -> 0.1uF
- C7: value 10mkF -> 10uF
- D1: value DIODE_BRIDGE -> DB104
- Q1: value (none) -> STP14NM50N; device my_devices:TRANSISTOR_NPN -> my_devices:MOSFET_N
- Q2: value (none) -> 2N3904
- Q3, Q7: value (none) -> 2N3906BU
- Q8: value MOSFET_N -> STP14NM50N
- R5, R8: value R -> 600
- R6, R7: value R -> 39K
- U2: value 5V -> L4940V5
- U3: value 3V3 -> L78L33ACZ-AP
Connections:
- new net N$17: C8.P$1, R10.P$1, U6.CKIN
- new net N$18: C9.P$1, U6.IGND
- new net N$19: C10.P$1, U6.IN
- new net N$20: BM1.P$2, C10.P$2
- new net N$24: C11.P$2, IC1.XTAL2, X1.P$2
- new net N$25: C13.P$1, L1.L2-2
- new net N$26: C12.P$2, IC1.XTAL1, X1.P$1
- new net N$27: C13.P$2, L1.L2-1
- new net N$28: C14.P$2, L2.L2-1
- new net N$29: C14.P$1, L2.L2-2
- new net N$32: J1.VCC, Q2.B, R15.P$1, SW1.P$2
- new net NOISE_LEVEL: IC1.(ADC1)PA1, U6.OUT
- new net NOISE_RESET: IC1.(MOSI)PB5, U6.RESET
- new net NOISE_STROBE: IC1.(SS)PB4, U6.STROBE
- new net TRANSMITTER: IC1.(MISO)PB6, U7.GND
- net +5V: now also L1.L1-2; no longer U$1.P$2
- net GND: now also Q1.S, Q9.S, R14.P$1, R15.P$2; no longer J1.GND
- net I2C_SCL: now also U4.SCL, U5.SCL
- net I2C_SDA: now also U4.SDA, U5.SDA
- net N$13: now also L1.L1-3; no longer U$1.P$1
- net N$14: now also L2.L1-1; no longer U$2.P$2
- net N$15: now also L2.L1-2; no longer U$2.P$1
- net N$16: now also R9.P$1; no longer R9.P$2
- net N$2: now also J1.GND, Q1.D; no longer J1.VCC, Q1.E
- net N$3: now also Q1.G, R14.P$2; no longer Q1.B
- net N$4: now also L1.L1-1, Q9.D; no longer Q1.C, Q2.B, SW1.P$2
- net N$9: now also Q9.G
- net OUTDOOR_+5V: now also R10.P$2, R9.P$2, U6.VCC, U7.VCC; no longer R9.P$1
- net OUTDOOR_3V3: now also U4.VIN, U5.VCC
- net OUTDOOR_GND: now also BM1.P$1, C11.P$1, C12.P$1, C8.P$2, C9.P$2, U4.GND, U5.GND, U6.GND, U7.DATA
Other:
- note added: "30 turns"
- note added: "45 turns"
- note added: "https://cxem.net/sound/light/light82.php"
- note added: "https://habr.com/ru/post/491530/"
- note added: "~18..23 turns"
- moved on the sheet: ACDC1, C3, C4, C5, D1, J1, Q8, R1, R2, R4, R5, R6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

Commit message: Commit schematics for a window control project
Parts:
- removed C5: 1000uF, my_devices:C
- added B1: HALL_SENSOR, my_devices:HALL_SENSOR
- added R16: 4 om / 5W, my_devices:R
- added R17, R18: 10K, my_devices:R
- added SW2: SWITCH, my_devices:SWITCH
- C1: value K10-17B (1000pF) -> 100 pF; device my_devices:C -> my_devices:C-1
- C10: value 0.01uF -> 0.01 uF
- C11, C12: value 22pF -> 22 pF
- C13, C14: value 10pF -> 0.47 uF / 20V
- C2: value K10-17B (1000pF) -> 1000 uF
- C3, C4: value 1000uF -> 1000 uF
- C6: value 0.1uF -> 0.1 uF
- C7: value 10uF -> 10 uF
- C8: value 33pF -> 33 pF
- C9: value 0.01uF -> 0.1 uF
- Q3: value 2N3906BU -> 2N3904; device my_devices:TRANSISTOR_PNP -> my_devices:TRANSISTOR_NPN
- R1, R11, R12, R13, R4: value 600 -> 620
- R2: value 600 -> 400
- R5: value 600 -> 10K
- R6, R7: value 39K -> 620
- R8: value 600 -> 2K; device my_devices:R -> my_devices:RD
- U3: value L78L33ACZ-AP -> CD4047; device my_devices:VOLTAGE_REGULATOR -> my_devices:CD4047
- U5: value BMP280 -> BMP280 / 5V
Connections:
- removed net OUTDOOR_3V3: C5.PIN_PLUS, U3.OUT, U4.VIN, U5.VCC
- new net +5V_GEN: C2.PIN_PLUS, R16.P$1, SW2.P$2, U3.-TRG, U3.AST, U3.AST_, U3.VCC
- new net HALL_OUT: Q3.C, Q7.B, R18.P$1, U1.IO4
- new net N$30: Q9.G, R7.P$2
- new net N$31: R7.P$1, U3.Q
- new net N$33: R6.P$1, U3.Q_
- new net N$34: R8.P1, U3.R
- new net N$35: L1.L1-2, R16.P$2
- new net N$37: B1.OUT, Q3.B, R17.P$1
- new net N$38: Q1.G, Q7.C, R14.P$2
- net +5V: now also B1.VCC, R17.P$2, SW2.P$1; no longer L1.L1-2, R5.P$2, R6.P$2, R7.P$2, R8.P$2
- net 3V3: now also R18.P$2
- net GND: now also B1.GND, C2.PIN_GND, U3.+TRG, U3.EXT_RESET, U3.GND, U3.RE_TRG; no longer Q7.C
- net N$10: now also R5.P$2, R8.P2, R8.P3; no longer C2.PIN_GND, Q3.C, Q8.G, R8.P$1
- net N$11: now also C1.P$2, U3.C; no longer C1.PIN_PLUS, Q3.B, R6.P$1
- net N$12: now also Q8.G, R6.P$2; no longer C2.PIN_PLUS, Q7.B, R7.P$1
- net N$3: now also Q7.E; no longer Q1.G, R14.P$2
- net N$9: now also C1.P$1, U3.RC; no longer C1.PIN_GND, Q7.E, Q9.G
- net OUTDOOR_+5V: now also U4.VIN, U5.VCC; no longer U3.IN
- net OUTDOOR_GND: no longer C5.PIN_GND, U3.GND
Other:
- note added: "1.1 uH"
- note added: "10 turns"
- note added: "15-20 turns"
- note added: "5V Module required!"
- note added: "Freq ~ 200 KHz"
- note added: "calc L -> https://coil32.ru/calc/ferrite-rod.html"
- note added: "calc LC -> https://coil32.ru/calc/jslcc.html"
- note added: "~8..13 turns 1.347 uH"
- note removed: "30 turns"
- note removed: "45 turns"
- note removed: "~18..23 turns"
- moved on the sheet: BM1, C10, C13, C14, C2, C8, C9, J1, Q1, Q2, Q3, Q7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

Commit message: Changed some nomanals during making order
Parts:
- removed C14: 0.47 uF / 20V, my_devices:C-1
- added C5: 10 uF, my_devices:C
- B1: value HALL_SENSOR -> A3144
- C10: value 0.01 uF -> 33 pF
- C11: value 22 pF -> 0.47 uF / 20V
- C12: value 22 pF -> 1000 uF; device my_devices:C-1 -> my_devices:C
- C13: value 0.47 uF / 20V -> 1000 uF; device my_devices:C-1 -> my_devices:C; SPICEPREFIX C -> (none)
- C2, C3: value 1000 uF -> 22 pF; device my_devices:C -> my_devices:C-1
- C6: value 0.1 uF -> 0.22 uF
- C7: value 10 uF -> 0.47 uF / 20V; device my_devices:C -> my_devices:C-1; SPICEPREFIX (none) -> C
- C8: value 33 pF -> 0.01 uF
- D1: value DB104 -> RGBLED; device my_devices:DIODE_BRIDGE -> my_devices:RGBLED
- D2: value RGBLED -> DB104; device my_devices:RGBLED -> my_devices:DIODE_BRIDGE
- J1: value SERVO -> MTR-SERVO-FS5103B
- Q1: value STP14NM50N -> 2N3904; device my_devices:MOSFET_N -> my_devices:TRANSISTOR_NPN
- Q6: value 2N3904 -> 2N3906BU; device my_devices:TRANSISTOR_NPN -> my_devices:TRANSISTOR_PNP
- Q7: value 2N3906BU -> STP14NM50N; device my_devices:TRANSISTOR_PNP -> my_devices:MOSFET_N
- R10: value 200k -> 10K
- R11, R12, R4: value 620 -> 10K
- R13: value 620 -> 2K; device my_devices:R -> my_devices:RD
- R15, R3, R5: value 10K -> 620
- R16: value 4 om / 5W -> 620
- R17: value 10K -> 4 om / 5W
- R18: value 10K -> 200k
- R2: value 400 -> 620
- R8: value 2K -> 10K; device my_devices:RD -> my_devices:R
- U2: value L4940V5 -> CD4047; device my_devices:VOLTAGE_REGULATOR -> my_devices:CD4047
- U3: value CD4047 -> BMP280 / 5V; device my_devices:CD4047 -> my_devices:BME280
- U4: value GY-SGP30 -> MSGEQ7; device my_devices:GY-SGP30 -> my_devices:MSGEQ7
- U5: value BMP280 / 5V -> KIA7805API-U/PF; device my_devices:BME280 -> my_devices:VOLTAGE_REGULATOR
- U6: value MSGEQ7 -> GY-SGP30; device my_devices:MSGEQ7 -> my_devices:GY-SGP30
Connections:
- net +5V: now also Q1.C, Q2.C, Q3.C, R11.P$2; no longer Q4.C, Q5.C, Q6.C, R17.P$2
- net +5V_GEN: now also C4.PIN_PLUS, R17.P$1, U2.-TRG, U2.AST, U2.AST_, U2.VCC; no longer C2.PIN_PLUS, R16.P$1, U3.-TRG, U3.AST, U3.AST_, U3.VCC
- net 3V3: now also Q4.C, R8.P$2; no longer Q2.C, R18.P$2
- net GND: now also C4.PIN_GND, D1.GND, Q5.E, Q7.S, R10.P$2, R4.P$1, R9.P$2, U2.+TRG, U2.EXT_RESET, U2.GND, U2.RE_TRG; no longer C2.PIN_GND, D2.GND, Q1.S, Q3.E, R14.P$1, R15.P$2, R3.P$2, U3.+TRG, U3.EXT_RESET, U3.GND, U3.RE_TRG
- net GPIO_RGB_B: now also R1.P$1; no longer R11.P$1
- net GPIO_RGB_G: now also R2.P$1; no longer R12.P$1
- net GPIO_RGB_R: now also R3.P$1; no longer R13.P$1
- net GPIO_SERVO_EN: now also R6.P$1; no longer R2.P$1
- net GPIO_SERVO_IS_ON: now also R5.P$1; no longer R4.P$1
- net GPIO_SERVO_PULSE: now also R7.P$1; no longer R1.P$1
- net HALL_OUT: now also Q5.C, Q6.B, R8.P$1; no longer Q3.C, Q7.B, R18.P$1
- net I2C_SCL: now also U3.SCL, U6.SCL; no longer U4.SCL, U5.SCL
- net I2C_SDA: now also U3.SDA, U6.SDA; no longer U4.SDA, U5.SDA
- net N$1: now also R7.P$2; no longer R1.P$2
- net N$10: now also R12.P$2, R13.P2, R13.P3; no longer R5.P$2, R8.P2, R8.P3
- net N$11: now also U2.C; no longer U3.C
- net N$12: now also R15.P$2; no longer R6.P$2
- net N$14: now also D2.AC1; no longer D1.AC1
- net N$15: now also D2.AC2; no longer D1.AC2
- net N$16: now also C5.PIN_PLUS, R14.P$1; no longer C7.PIN_PLUS, R9.P$1
- net N$17: now also C10.P$1, R18.P$1, U4.CKIN; no longer C8.P$1, R10.P$1, U6.CKIN
- net N$18: now also U4.IGND; no longer U6.IGND
- net N$19: now also C8.P$1, U4.IN; no longer C10.P$1, U6.IN
- net N$2: now also Q7.D; no longer Q1.D
- net N$20: now also C8.P$2; no longer C10.P$2
- net N$21: now also Q1.B, R1.P$2; no longer Q4.B, R11.P$2
- net N$22: now also Q2.B, R2.P$2; no longer Q5.B, R12.P$2
- net N$23: now also Q3.B, R3.P$2; no longer Q6.B, R13.P$2
- net N$24: now also C2.P$2; no longer C11.P$2
- net N$25: now also C7.P$2; no longer C13.P$2
- net N$26: now also C3.P$2; no longer C12.P$2
- net N$27: now also C7.P$1; no longer C13.P$1
- net N$28: now also C11.P$2; no longer C14.P$2
- net N$29: now also C11.P$1; no longer C14.P$1
- net N$3: now also Q6.E, R6.P$2; no longer Q7.E, R2.P$2
- net N$30: now also R16.P$2; no longer R7.P$2
- net N$31: now also R16.P$1, U2.Q; no longer R7.P$1, U3.Q
- net N$32: now also Q4.B, R10.P$1; no longer Q2.B, R15.P$1
- net N$33: now also R15.P$1, U2.Q_; no longer R6.P$1, U3.Q_
- net N$34: now also R13.P1, U2.R; no longer R8.P1, U3.R
- net N$35: now also R17.P$2; no longer R16.P$2
- net N$37: now also Q5.B, R11.P$1; no longer Q3.B, R17.P$1
- net N$38: now also Q6.C, Q7.G, R4.P$2; no longer Q1.G, Q7.C, R14.P$2
- net N$5: now also D1.VIN_B, Q1.E; no longer D2.VIN_B, Q4.E
- net N$6: now also Q4.E, R5.P$2, R9.P$1; no longer Q2.E, R3.P$1, R4.P$2
- net N$7: now also D1.VIN_G, Q2.E; no longer D2.VIN_G, Q5.E
- net N$8: now also D1.VIN_R, Q3.E; no longer D2.VIN_R, Q6.E
- net N$9: now also R12.P$1, U2.RC; no longer R5.P$1, U3.RC
- net NOISE_LEVEL: now also U4.OUT; no longer U6.OUT
- net NOISE_RESET: now also U4.RESET; no longer U6.RESET
- net NOISE_STROBE: now also U4.STROBE; no longer U6.STROBE
- net OUTDOOR_+5V: now also C13.PIN_PLUS, R14.P$2, R18.P$2, U3.VCC, U4.VCC, U5.OUT, U6.VIN; no longer C4.PIN_PLUS, R10.P$2, R9.P$2, U2.OUT, U4.VIN, U5.VCC, U6.VCC
- net OUTDOOR_GND: now also C10.P$2, C12.PIN_GND, C13.PIN_GND, C2.P$1, C3.P$1, C5.PIN_GND, D2.GND, U3.GND; no longer C11.P$1, C12.P$1, C3.PIN_GND, C4.PIN_GND, C7.PIN_GND, C8.P$2, D1.GND, U2.GND
- net VCC: now also C12.PIN_PLUS, D2.VCC, U5.IN; no longer C3.PIN_PLUS, D1.VCC, U2.IN
Other:
- moved on the sheet: C10, C11, C4, C8, Q2, Q3, Q4, Q5, Q6, R1, R10, R11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

Commit message: added fan_pwm driver
Parts:
- removed Q7: STP14NM50N, my_devices:MOSFET_N
- added C14, C16: 10 uF, my_devices:C
- added C15: 3 nF ?, my_devices:C-1
- added C17, C20: C-1, my_devices:C-1
- added C18: 10uF, my_devices:C
- added C19: 1 nF, my_devices:C-1
- added D3, D4, D6: SB560, my_devices:D_SCHOTTKY
- added D5, D8: BAT41, my_devices:D_SCHOTTKY
- added D7, D9: 1N4001, my_devices:D
- added L3, L4: 1000 uH, my_devices:L
- added Q10, Q12, Q16: 2N3906BU, my_devices:TRANSISTOR_PNP
- added Q11, Q13, Q14: 2N3904, my_devices:TRANSISTOR_NPN
- added Q17: STP14NM50N, my_devices:MOSFET_N
- added R19: 620, my_devices:R
- added R21, R23: 10K, my_devices:R
- added U8: NE555P, my_devices:NE555P
- added U9: SN74LS32N, my_devices:SN74LS32N
- C11: value 0.47 uF / 20V -> C-1
- C7: value 0.47 uF / 20V -> 3 nF ?; SPICEPREFIX C -> (none)
- J1: value MTR-SERVO-FS5103B -> SERVO
- L1: value L-3 -> ~6 uH; device my_devices:L-3 -> my_devices:L-4
- L2: value L-2 -> L; device my_devices:L-2 -> my_devices:L
- Q6: value 2N3906BU -> (none)
- R10, R12, R9: value 10K -> 620
- R13: value 2K -> 10K
- R15: value 620 -> 5K / 125 mW
- R16: value 620 -> R
- R17: value 4 om / 5W -> 10K
- R5: value 620 -> 10K
- R6: value 620 -> 4K
- R7: value 620 -> RD; device my_devices:R -> my_devices:RD
- R8: value 10K -> R
Connections:
- removed net GPIO_SERVO_EN: R6.P$1, U1.IO18
- removed net GPIO_SERVO_IS_ON: R5.P$1, U1.IO21
- removed net GPIO_SERVO_PULSE: R7.P$1, U1.IO19
- removed net HALL_OUT: Q5.C, Q6.B, R8.P$1, U1.IO4
- removed net N$37: B1.OUT, Q5.B, R11.P$1
- new net HALL_OUT_INV: B1.OUT, R11.P$1, R19.P$2, U9.1A
- new net N$39: D8.P$1, L4.P$2, Q4.C
- new net N$40: J1.VCC, Q17.S
- new net N$41: Q10.B, Q11.B, U2.Q_
- new net N$42: Q12.B, Q13.B, U2.Q
- new net N$43: C18.PIN_PLUS, Q16.C, R4.P$1, R8.P$2, U8.RESET, U8.VCC
- new net N$44: C19.P$1, U8.CONT
- new net N$45: Q14.B, U2.OSC_OUT
- new net N$46: C20.P$2, D7.P$2, D9.P$1, U8.THRES, U8.TRIG
- new net N$47: D7.P$1, R7.P3, U8.DISCH
- new net N$48: D9.P$2, R7.P2
- new net N$49: R7.P1, R8.P$1
- new net N$50: J1.PULSE, Q5.C, R16.P$2
- new net N$51: C16.PIN_PLUS, D8.P$2, Q17.G, R6.P$2
- new net N$52: Q6.B, R17.P$1, U8.OUT
- new net SERVO_ENABLE_INV: R10.P$2, U9.1B
- new net SERVO_IS_ENABLED_INV: R12.P$2
- new net SERVO_PWM: R9.P$2, U9.3A
- new net SERVO_PWM_CONTROL: C17.P$2, Q5.B, R23.P$1, U9.3Y
- net +5V: now also L4.P$1, Q16.E, Q17.D, Q6.E, R16.P$1, R17.P$2, R21.P$1, R23.P$2, U9.VCC; no longer SW1.P$1
- net +5V_GEN: now also D6.P$1, L3.P$1; no longer R17.P$1
- net 3V3: no longer Q4.C, R8.P$2
- net GND: now also C14.PIN_GND, C16.PIN_GND, C18.PIN_GND, C19.P$2, C20.P$1, J1.GND, Q10.C, Q12.C, Q14.E, Q4.E, R15.P$1, R4.P$2, R5.P$1, R6.P$1, SW1.P$1, U8.GND, U9.GND; no longer Q7.S, R10.P$2, R4.P$1, R9.P$2
- net N$1: now also U9.1Y, U9.2B; no longer J1.PULSE, R7.P$2
- net N$10: now also C1.P$1, U2.RC; no longer R12.P$2
- net N$12: now also Q10.E, Q11.E; no longer R15.P$2
- net N$13: now also D3.P$2; no longer L1.L1-3
- net N$14: now also C11.P$2, L2.P$2; no longer L2.L1-1
- net N$15: now also C11.P$1, L2.P$1; no longer L2.L1-2
- net N$2: now also SW1.P$2, U9.2A; no longer J1.GND, Q7.D
- net N$25: now also D3.P$1, L1.P$1; no longer L1.L2-1
- net N$27: now also C15.P$2, D6.P$2, L1.P$2; no longer L1.L2-2
- net N$28: now also R10.P$1, U1.IO21; no longer C11.P$2, L2.L2-1
- net N$29: now also R12.P$1, U1.IO18; no longer C11.P$1, L2.L2-2
- net N$3: now also U9.2Y, U9.3B; no longer Q6.E, R6.P$2
- net N$30: now also C14.PIN_PLUS, D5.P$2, Q11.C, Q13.C, R15.P$2; no longer Q9.G, R16.P$2
- net N$31: now also C15.P$1, D4.P$1, L1.P$3; no longer R16.P$1, U2.Q
- net N$32: now also R19.P$1, U1.IO16; no longer J1.VCC, Q4.B, R10.P$1, SW1.P$2
- net N$33: now also Q12.E, Q13.E, Q9.G; no longer R15.P$1, U2.Q_
- net N$35: now also Q4.B, Q6.C, R5.P$2; no longer L1.L1-2, R17.P$2
- net N$38: now also C17.P$1, Q16.B, R21.P$2; no longer Q6.C, Q7.G, R4.P$2
- net N$4: now also D4.P$2; no longer L1.L1-1
- net N$6: now also U1.IO19; no longer Q4.E, R5.P$2
- net N$9: now also D5.P$1, L3.P$2, Q14.C; no longer C1.P$1, R12.P$1, U2.RC
Other:
- note added: "Freq ~ Q: 225 KHz OSC OUT: 450 KHz"
- note added: "https://vip-cxema.org/index.php/online-raschjoty/366-raschjot-povyshayushchego-dc-dc-preobrazovatelya"
- note added: "~15-20V max 50 mA"
- note removed: "1.1 uH"
- note removed: "10 turns"
- note removed: "15-20 turns"
- note removed: "Freq ~ 200 KHz"
- note removed: "~8..13 turns 1.347 uH"
- moved on the sheet: B1, C11, C12, C13, C7, D2, J1, Q4, Q5, Q6, Q8, Q9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
